Commit message: publish gripper position via hardware interface

File: xarm_description/urdf/xarm7/xarm7.ros2_control.xacro (robot description, xacro)
@@ -121,4 +121,9 @@
         <!-- <state_interface name="effort"/> -->
       </joint>
+      <xacro:if value="${add_gripper}">
+        <joint name="${prefix}drive_joint">
+          <state_interface name="position"/>
+        </joint>
+      </xacro:if>
     </ros2_control>
   </xacro:macro>

Commit message: publish gripper position via hardware interface

File: xarm_description/urdf/xarm7/xarm7.ros2_control.xacro (robot description, xacro)
@@ -121,4 +121,10 @@
         <!-- <state_interface name="effort"/> -->
       </joint>
+      <xacro:if value="${add_gripper}">
+        <joint name="${prefix}drive_joint">
+          <state_interface name="position"/>
+          <state_interface name="velocity"/>
+        </joint>
+      </xacro:if>
     </ros2_control>
   </xacro:macro>
