Commit message: simplify arm mesh

File: xarm_description/urdf/xarm7/xarm7.urdf.xacro (robot description, xacro)
@@ -23,7 +23,7 @@
     <xacro:unless value="${model_num >= 1305 and model_num != 1380}">
       <xacro:property name="visual_dir" value="xarm7/visual"/>
-      <xacro:property name="collision_dir" value="xarm7/visual"/>
+      <xacro:property name="collision_dir" value="xarm7/collision"/>
       <xacro:property name="add_mesh_suffix" value="true"/>
-      <xacro:property name="collison_mesh_suffix" value="stl"/>
+      <xacro:property name="collison_mesh_suffix" value="STL"/>
       <xacro:if value="${model_num >= 1300}">
         <xacro:property name="link7_visual" value="end_tool/visual/end_tool_1300"/>
@@ -32,5 +32,5 @@
       <xacro:unless value="${model_num >= 1300}">
         <xacro:property name="link7_visual" value="xarm7/visual/link7"/>
-        <xacro:property name="link7_collision" value="end_tool/collision/end_tool"/>
+        <xacro:property name="link7_collision" value="xarm7/collision/link7"/>
       </xacro:unless>
     </xacro:unless>
