Commit message: adjustable is_ros2 value

File: xarm_description/urdf/_private_macro.xacro (robot description, xacro)
@@ -1,5 +1,5 @@
 <?xml version='1.0' encoding='utf-8'?>
 <robot xmlns:xacro="http://ros.org/wiki/xacro" name="private_macro">
-  <xacro:property name="is_ros2" value="true" scope="parent"/>
+  <xacro:property name="is_ros2" default="true"/>
   <xacro:property name="use_xacro_load_yaml" value="true" scope="parent"/>
   <xacro:property name="use_len" value="true" scope="parent"/>
