Commit message: added collision shpere macro

File: xarm_description/urdf/common/common.link.xacro (robot description, xacro)
@@ -61,4 +61,12 @@
     </collision>
   </xacro:macro>
+  <xacro:macro name="common_link_sphere_collision" params="name radius:='0.0' xyz='0 0 0'">
+    <collision name="${name}">
+      <origin xyz="${xyz}" rpy="0 0 0"/>
+      <geometry>
+        <sphere radius="${radius}"/>
+      </geometry>
+    </collision>
+  </xacro:macro>
   <xacro:macro name="common_joint_origin" params="joint_kinematic_params">
     <origin xyz="${joint_kinematic_params['x']} ${joint_kinematic_params['y']} ${joint_kinematic_params['z']}" rpy="${joint_kinematic_params['roll']} ${joint_kinematic_params['pitch']} ${joint_kinematic_params['yaw']}" />
