Commit message: simplify gripper mesh

File: xarm_description/urdf/gripper/xarm_gripper.urdf.xacro (robot description, xacro)
@@ -22,8 +22,16 @@
         origin_rpy="0 0 0"
         material_name="${prefix}White" />
-      <xacro:common_link_collision
-        mesh_filename="gripper/xarm/base_link"
-        origin_xyz="0 0 0"
-        origin_rpy="0 0 0" />
+      <collision>
+        <origin xyz="-0.0015 0 0.055" rpy="0 0 0"/>
+        <geometry>
+          <box size="0.053 0.1 0.1"/>
+        </geometry>
+      </collision>
+      <collision>
+        <origin xyz="0.03 -0.062 0.025" rpy="0 0 0"/>
+        <geometry>
+          <box size="0.076 0.024 0.04"/>
+        </geometry>
+      </collision>
     </link>
     <link name="${prefix}left_outer_knuckle">
@@ -40,8 +48,10 @@
         origin_rpy="0 0 0"
         material_name="${prefix}Silver" />
-      <xacro:common_link_collision
-        mesh_filename="gripper/xarm/left_outer_knuckle"
-        origin_xyz="0 0 0"
-        origin_rpy="0 0 0" />
+      <collision>
+        <origin xyz="0 0.015 0.02" rpy="0.48 0 0"/>
+        <geometry>
+          <box size="0.012 0.069 0.033"/>
+        </geometry>
+      </collision>
     </link>
     <joint name="${prefix}drive_joint" type="revolute">
@@ -65,8 +75,22 @@
         origin_rpy="0 0 0"
         material_name="${prefix}Silver" />
-      <xacro:common_link_collision
-        mesh_filename="gripper/xarm/left_finger"
-        origin_xyz="0 0 0"
-        origin_rpy="0 0 0" />
+      <collision>
+        <origin xyz="0 -0.0224 0.04" rpy="0 0 0"/>
+        <geometry>
+          <box size="0.032 0.0072 0.042"/>
+        </geometry>
+      </collision>
+      <collision>
+        <origin xyz="0 -0.0154 0.036" rpy="0 0 0"/>
+        <geometry>
+          <box size="0.032 0.0068 0.034"/>
+        </geometry>
+      </collision>
+      <collision>
+        <origin xyz="0 -0.008 0.008" rpy="0.8 0 0"/>
+        <geometry>
+          <box size="0.016 0.012 0.036"/>
+        </geometry>
+      </collision>
     </link>
     <joint name="${prefix}left_finger_joint" type="revolute">
@@ -91,8 +115,10 @@
         origin_rpy="0 0 0"
         material_name="${prefix}Silver" />
-      <xacro:common_link_collision
-        mesh_filename="gripper/xarm/left_inner_knuckle"
-        origin_xyz="0 0 0"
-        origin_rpy="0 0 0" />
+      <collision>
+        <origin xyz="0 0.016 0.02" rpy="-0.7 0 0"/>
+        <geometry>
+          <box size="0.027 0.012 0.061"/>
+        </geometry>
+      </collision>
     </link>
     <joint name="${prefix}left_inner_knuckle_joint" type="revolute">
@@ -117,8 +143,10 @@
         origin_rpy="0 0 0"
         material_name="${prefix}Silver" />
-      <xacro:common_link_collision
-        mesh_filename="gripper/xarm/right_outer_knuckle"
-        origin_xyz="0 0 0"
-        origin_rpy="0 0 0" />
+      <collision>
+        <origin xyz="0 -0.015 0.02" rpy="-0.48 0 0"/>
+        <geometry>
+          <box size="0.012 0.069 0.033"/>
+        </geometry>
+      </collision>
     </link>
     <joint name="${prefix}right_outer_knuckle_joint" type="revolute">
@@ -143,8 +171,22 @@
         origin_rpy="0 0 0"
         material_name="${prefix}Silver" />
-      <xacro:common_link_collision
-        mesh_filename="gripper/xarm/right_finger"
-        origin_xyz="0 0 0"
-        origin_rpy="0 0 0" />
+      <collision>
+        <origin xyz="0 0.0224 0.04" rpy="0 0 0"/>
+        <geometry>
+          <box size="0.032 0.0072 0.042"/>
+        </geometry>
+      </collision>
+      <collision>
+        <origin xyz="0 0.0154 0.036" rpy="0 0 0"/>
+        <geometry>
+          <box size="0.032 0.0068 0.034"/>
+        </geometry>
+      </collision>
+      <collision>
+        <origin xyz="0 0.008 0.008" rpy="-0.8 0 0"/>
+        <geometry>
+          <box size="0.016 0.012 0.036"/>
+        </geometry>
+      </collision>
     </link>
     <joint name="${prefix}right_finger_joint" type="revolute">
@@ -169,8 +211,10 @@
         origin_rpy="0 0 0"
         material_name="${prefix}Silver" />
-      <xacro:common_link_collision
-        mesh_filename="gripper/xarm/right_inner_knuckle"
-        origin_xyz="0 0 0"
-        origin_rpy="0 0 0" />
+      <collision>
+        <origin xyz="0 -0.016 0.02" rpy="0.7 0 0"/>
+        <geometry>
+          <box size="0.027 0.012 0.061"/>
+        </geometry>
+      </collision>
     </link>
     <joint name="${prefix}right_inner_knuckle_joint" type="revolute">

Commit message: Fix to switch finger_extension

File: xarm_description/urdf/gripper/xarm_gripper.urdf.xacro (robot description, xacro)
@@ -1,5 +1,5 @@
 <?xml version="1.0"?>
 <robot xmlns:xacro="http://ros.org/wiki/xacro" name="xarm_gripper">
-  <xacro:macro name="xarm_gripper_urdf" params="prefix:='' attach_to:='' attach_xyz:='0 0 0' attach_rpy:='0 0 0' ">
+  <xacro:macro name="xarm_gripper_urdf" params="prefix:='' attach_to:='' attach_xyz:='0 0 0' attach_rpy:='0 0 0' use_default_finger_extension:='true' ">
     <xacro:unless value="${attach_to == ''}">
       <joint name="${prefix}gripper_fix" type="fixed">
@@ -28,10 +28,4 @@
         </geometry>
       </collision>
-      <collision>
-        <origin xyz="0.03 -0.062 0.025" rpy="0 0 0"/>
-        <geometry>
-          <box size="0.076 0.024 0.04"/>
-        </geometry>
-      </collision>
     </link>
     <link name="${prefix}left_outer_knuckle">
@@ -75,10 +69,4 @@
         origin_rpy="0 0 0"
         material_name="${prefix}Silver" />
-      <collision>
-        <origin xyz="0 -0.0224 0.04" rpy="0 0 0"/>
-        <geometry>
-          <box size="0.032 0.0072 0.042"/>
-        </geometry>
-      </collision>
       <collision>
         <origin xyz="0 -0.0154 0.036" rpy="0 0 0"/>
@@ -172,10 +160,4 @@
         material_name="${prefix}Silver" />
       <collision>
-        <origin xyz="0 0.0224 0.04" rpy="0 0 0"/>
-        <geometry>
-          <box size="0.032 0.0072 0.042"/>
-        </geometry>
-      </collision>
-      <collision>
         <origin xyz="0 0.0154 0.036" rpy="0 0 0"/>
         <geometry>
@@ -232,4 +214,13 @@
       <child link="${prefix}link_tcp" />
     </joint>
+    <xacro:if value="${use_default_finger_extension}">
+      <xacro:include filename="$(find xarm_description)/urdf/gripper/finger_extension.xacro"/>
+      <xacro:finger_extension name="${prefix}left" parent="${prefix}left_finger">
+        <origin rpy="0 0 0" xyz="0 -0.0225 0.037"/>
+      </xacro:finger_extension>
+      <xacro:finger_extension name="${prefix}right" parent="${prefix}right_finger">
+        <origin rpy="0 0 0" xyz="0 0.0225 0.037"/>
+      </xacro:finger_extension>
+    </xacro:if>
   </xacro:macro>
 </robot>

Commit message: Fix size of collision box

File: xarm_description/urdf/gripper/xarm_gripper.urdf.xacro (robot description, xacro)
@@ -72,5 +72,5 @@
         <origin xyz="0 -0.0154 0.036" rpy="0 0 0"/>
         <geometry>
-          <box size="0.032 0.0068 0.034"/>
+          <box size="0.016 0.0068 0.034"/>
         </geometry>
       </collision>
@@ -162,5 +162,5 @@
         <origin xyz="0 0.0154 0.036" rpy="0 0 0"/>
         <geometry>
-          <box size="0.032 0.0068 0.034"/>
+          <box size="0.016 0.0068 0.034"/>
         </geometry>
       </collision>

Commit message: Rename finger_extension to finger_tip

File: xarm_description/urdf/gripper/xarm_gripper.urdf.xacro (robot description, xacro)
@@ -1,5 +1,5 @@
 <?xml version="1.0"?>
 <robot xmlns:xacro="http://ros.org/wiki/xacro" name="xarm_gripper">
-  <xacro:macro name="xarm_gripper_urdf" params="prefix:='' attach_to:='' attach_xyz:='0 0 0' attach_rpy:='0 0 0' use_default_finger_extension:='true' ">
+  <xacro:macro name="xarm_gripper_urdf" params="prefix:='' attach_to:='' attach_xyz:='0 0 0' attach_rpy:='0 0 0' use_default_finger_tip:='true' ">
     <xacro:unless value="${attach_to == ''}">
       <joint name="${prefix}gripper_fix" type="fixed">
@@ -214,12 +214,12 @@
       <child link="${prefix}link_tcp" />
     </joint>
-    <xacro:if value="${use_default_finger_extension}">
-      <xacro:include filename="$(find xarm_description)/urdf/gripper/finger_extension.xacro"/>
-      <xacro:finger_extension name="${prefix}left" parent="${prefix}left_finger">
+    <xacro:if value="${use_default_finger_tip}">
+      <xacro:include filename="$(find xarm_description)/urdf/gripper/finger_tip.xacro"/>
+      <xacro:finger_tip name="${prefix}left" parent="${prefix}left_finger">
         <origin rpy="0 0 0" xyz="0 -0.0225 0.037"/>
-      </xacro:finger_extension>
-      <xacro:finger_extension name="${prefix}right" parent="${prefix}right_finger">
+      </xacro:finger_tip>
+      <xacro:finger_tip name="${prefix}right" parent="${prefix}right_finger">
         <origin rpy="0 0 0" xyz="0 0.0225 0.037"/>
-      </xacro:finger_extension>
+      </xacro:finger_tip>
     </xacro:if>
   </xacro:macro>

Commit message: added gripper collision sphere

File: xarm_description/urdf/gripper/xarm_gripper.urdf.xacro (robot description, xacro)
@@ -1,5 +1,5 @@
 <?xml version="1.0"?>
 <robot xmlns:xacro="http://ros.org/wiki/xacro" name="xarm_gripper">
-  <xacro:macro name="xarm_gripper_urdf" params="prefix:='' attach_to:='' attach_xyz:='0 0 0' attach_rpy:='0 0 0' use_default_finger_tip:='true' ">
+  <xacro:macro name="xarm_gripper_urdf" params="prefix:='' attach_to:='' attach_xyz:='0 0 0' attach_rpy:='0 0 0' use_default_finger_tip:='true' use_collision_sphere:='false' ">
     <xacro:unless value="${attach_to == ''}">
       <joint name="${prefix}gripper_fix" type="fixed">
@@ -22,10 +22,22 @@
         origin_rpy="0 0 0"
         material_name="${prefix}White" />
-      <collision>
-        <origin xyz="-0.0015 0 0.055" rpy="0 0 0"/>
-        <geometry>
-          <box size="0.053 0.1 0.1"/>
-        </geometry>
-      </collision>
+      <xacro:unless value="${use_collision_sphere}">
+        <collision>
+          <origin xyz="-0.0015 0 0.055" rpy="0 0 0"/>
+          <geometry>
+            <box size="0.053 0.1 0.1"/>
+          </geometry>
+         </collision>
+      </xacro:unless>
+      <xacro:if value="${use_collision_sphere}">
+        <xacro:common_link_sphere_collision name="sphere1" xyz="0.005 -0.002 0.041" radius="0.04"/>
+        <xacro:common_link_sphere_collision name="sphere2" xyz="0.0 0.029 0.026" radius="0.04"/>
+        <xacro:common_link_sphere_collision name="sphere3" xyz="0.0 0.03 0.067" radius="0.04"/>
+        <xacro:common_link_sphere_collision name="sphere4" xyz="0.0 -0.037 0.023" radius="0.04"/>
+        <xacro:common_link_sphere_collision name="sphere5" xyz="0.0 -0.033 0.067" radius="0.04"/>
+        <xacro:common_link_sphere_collision name="sphere6" xyz="0.0 -0.004 0.067" radius="0.04"/>
+        <xacro:common_link_sphere_collision name="sphere7" xyz="0.021 -0.055 0.022" radius="0.03"/>
+        <xacro:common_link_sphere_collision name="sphere8" xyz="0.048 -0.053 0.025" radius="0.03"/>
+      </xacro:if>
     </link>
     <link name="${prefix}left_outer_knuckle">
@@ -42,10 +54,17 @@
         origin_rpy="0 0 0"
         material_name="${prefix}Silver" />
-      <collision>
-        <origin xyz="0 0.015 0.02" rpy="0.48 0 0"/>
-        <geometry>
-          <box size="0.012 0.069 0.033"/>
-        </geometry>
-      </collision>
+      <xacro:unless value="${use_collision_sphere}">
+        <collision>
+          <origin xyz="0 0.015 0.02" rpy="0.48 0 0"/>
+          <geometry>
+            <box size="0.012 0.069 0.033"/>
+          </geometry>
+        </collision>
+      </xacro:unless>
+      <xacro:if value="${use_collision_sphere}">
+        <xacro:common_link_sphere_collision name="sphere1" xyz="0.0 0.044 0.022" radius="0.01"/>
+        <xacro:common_link_sphere_collision name="sphere2" xyz="0.0 0.039 0.036" radius="0.01"/>
+        <xacro:common_link_sphere_collision name="sphere3" xyz="0.0 0.035 0.016" radius="0.01"/>
+      </xacro:if>
     </link>
     <joint name="${prefix}drive_joint" type="revolute">
@@ -69,16 +88,31 @@
         origin_rpy="0 0 0"
         material_name="${prefix}Silver" />
-      <collision>
-        <origin xyz="0 -0.0154 0.036" rpy="0 0 0"/>
-        <geometry>
-          <box size="0.016 0.0068 0.034"/>
-        </geometry>
-      </collision>
-      <collision>
-        <origin xyz="0 -0.008 0.008" rpy="0.8 0 0"/>
-        <geometry>
-          <box size="0.016 0.012 0.036"/>
-        </geometry>
-      </collision>
+      <xacro:unless value="${use_collision_sphere}">
+        <collision>
+          <origin xyz="0 -0.0154 0.036" rpy="0 0 0"/>
+          <geometry>
+            <box size="0.016 0.0068 0.034"/>
+          </geometry>
+        </collision>
+        <collision>
+          <origin xyz="0 -0.008 0.008" rpy="0.8 0 0"/>
+          <geometry>
+            <box size="0.016 0.012 0.036"/>
+          </geometry>
+        </collision>
+      </xacro:unless>
+      <xacro:if value="${use_collision_sphere}">
+        <xacro:common_link_sphere_collision name="sphere1" xyz="0.0 -0.005 0.005" radius="0.01"/>
+        <xacro:common_link_sphere_collision name="sphere2" xyz="0.0 -0.014 0.014" radius="0.01"/>
+        <xacro:common_link_sphere_collision name="sphere3" xyz="-0.009 -0.02 0.025" radius="0.01"/>
+        <xacro:common_link_sphere_collision name="sphere4" xyz="-0.009 -0.02 0.036" radius="0.01"/>
+        <xacro:common_link_sphere_collision name="sphere5" xyz="-0.009 -0.02 0.047" radius="0.01"/>
+        <xacro:common_link_sphere_collision name="sphere6" xyz="0.0 -0.02 0.025" radius="0.01"/>
+        <xacro:common_link_sphere_collision name="sphere7" xyz="0.009 -0.02 0.025" radius="0.01"/>
+        <xacro:common_link_sphere_collision name="sphere8" xyz="0.0 -0.02 0.036" radius="0.01"/>
+        <xacro:common_link_sphere_collision name="sphere9" xyz="0.0 -0.02 0.047" radius="0.01"/>
+        <xacro:common_link_sphere_collision name="sphere10" xyz="0.009 -0.02 0.036" radius="0.01"/>
+        <xacro:common_link_sphere_collision name="sphere11" xyz="0.009 -0.02 0.047" radius="0.01"/>
+      </xacro:if>
     </link>
     <joint name="${prefix}left_finger_joint" type="revolute">
@@ -103,10 +137,16 @@
         origin_rpy="0 0 0"
         material_name="${prefix}Silver" />
-      <collision>
-        <origin xyz="0 0.016 0.02" rpy="-0.7 0 0"/>
-        <geometry>
-          <box size="0.027 0.012 0.061"/>
-        </geometry>
-      </collision>
+      <xacro:unless value="${use_collision_sphere}">
+        <collision>
+          <origin xyz="0 0.016 0.02" rpy="-0.7 0 0"/>
+          <geometry>
+            <box size="0.027 0.012 0.061"/>
+          </geometry>
+        </collision>
+      </xacro:unless>
+      <xacro:if value="${use_collision_sphere}">
+        <xacro:common_link_sphere_collision name="sphere1" xyz="0.009 0.029 0.033" radius="0.01"/>
+        <xacro:common_link_sphere_collision name="sphere2" xyz="-0.009 0.029 0.033" radius="0.01"/>
+      </xacro:if>
     </link>
     <joint name="${prefix}left_inner_knuckle_joint" type="revolute">
@@ -131,10 +171,17 @@
         origin_rpy="0 0 0"
         material_name="${prefix}Silver" />
-      <collision>
-        <origin xyz="0 -0.015 0.02" rpy="-0.48 0 0"/>
-        <geometry>
-          <box size="0.012 0.069 0.033"/>
-        </geometry>
-      </collision>
+      <xacro:unless value="${use_collision_sphere}">
+        <collision>
+          <origin xyz="0 -0.015 0.02" rpy="-0.48 0 0"/>
+          <geometry>
+            <box size="0.012 0.069 0.033"/>
+          </geometry>
+        </collision>
+      </xacro:unless>
+      <xacro:if value="${use_collision_sphere}">
+        <xacro:common_link_sphere_collision name="sphere1" xyz="0.0 -0.044 0.022" radius="0.01"/>
+        <xacro:common_link_sphere_collision name="sphere2" xyz="0.0 -0.039 0.036" radius="0.01"/>
+        <xacro:common_link_sphere_collision name="sphere3" xyz="0.0 -0.035 0.016" radius="0.01"/>
+      </xacro:if>
     </link>
     <joint name="${prefix}right_outer_knuckle_joint" type="revolute">
@@ -165,10 +212,25 @@
         </geometry>
       </collision>
-      <collision>
-        <origin xyz="0 0.008 0.008" rpy="-0.8 0 0"/>
-        <geometry>
-          <box size="0.016 0.012 0.036"/>
-        </geometry>
-      </collision>
+      <xacro:unless value="${use_collision_sphere}">
+        <collision>
+          <origin xyz="0 0.008 0.008" rpy="-0.8 0 0"/>
+          <geometry>
+            <box size="0.016 0.012 0.036"/>
+          </geometry>
+        </collision>
+      </xacro:unless>
+      <xacro:if value="${use_collision_sphere}">
+        <xacro:common_link_sphere_collision name="sphere1" xyz="0.0 0.005 0.005" radius="0.01"/>
+        <xacro:common_link_sphere_collision name="sphere2" xyz="0.0 0.014 0.014" radius="0.01"/>
+        <xacro:common_link_sphere_collision name="sphere3" xyz="-0.009 0.02 0.025" radius="0.01"/>
+        <xacro:common_link_sphere_collision name="sphere4" xyz="-0.009 0.02 0.036" radius="0.01"/>
+        <xacro:common_link_sphere_collision name="sphere5" xyz="-0.009 0.02 0.047" radius="0.01"/>
+        <xacro:common_link_sphere_collision name="sphere6" xyz="0.0 0.02 0.025" radius="0.01"/>
+        <xacro:common_link_sphere_collision name="sphere7" xyz="0.009 0.02 0.025" radius="0.01"/>
+        <xacro:common_link_sphere_collision name="sphere8" xyz="0.0 0.02 0.036" radius="0.01"/>
+        <xacro:common_link_sphere_collision name="sphere9" xyz="0.0 0.02 0.047" radius="0.01"/>
+        <xacro:common_link_sphere_collision name="sphere10" xyz="0.009 0.02 0.036" radius="0.01"/>
+        <xacro:common_link_sphere_collision name="sphere11" xyz="0.009 0.02 0.047" radius="0.01"/>
+      </xacro:if>
     </link>
     <joint name="${prefix}right_finger_joint" type="revolute">
@@ -193,10 +255,16 @@
         origin_rpy="0 0 0"
         material_name="${prefix}Silver" />
-      <collision>
-        <origin xyz="0 -0.016 0.02" rpy="0.7 0 0"/>
-        <geometry>
-          <box size="0.027 0.012 0.061"/>
-        </geometry>
-      </collision>
+      <xacro:unless value="${use_collision_sphere}">
+        <collision>
+          <origin xyz="0 -0.016 0.02" rpy="0.7 0 0"/>
+          <geometry>
+            <box size="0.027 0.012 0.061"/>
+          </geometry>
+        </collision>
+      </xacro:unless>
+      <xacro:if value="${use_collision_sphere}">
+        <xacro:common_link_sphere_collision name="sphere1" xyz="-0.009 -0.029 0.033" radius="0.01"/>
+        <xacro:common_link_sphere_collision name="sphere2" xyz="0.009 -0.029 0.033" radius="0.01"/>
+      </xacro:if>
     </link>
     <joint name="${prefix}right_inner_knuckle_joint" type="revolute">
